Commit message: init

File: description/imu.xacro (robot description, xacro)
@@ -4,9 +4,9 @@
     <joint name="imu_joint" type="fixed">
         <parent link="chassis"/>
-        <child link="imu_link"/>
+        <child link="imu_l"/>
         <!-- Mount IMU near the center of the chassis -->
         <origin xyz=".18 0 0.03" rpy="0 0 0"/>
     </joint>
-    <link name="imu_link">
+    <link name="imu_l">
         <visual>
             <origin xyz="0 0 0" rpy="0 0 0"/>
@@ -25,5 +25,5 @@
         </collision>
     </link>
-    <gazebo reference="imu_link">
+    <gazebo reference="imu_l">
         <sensor name="imu_sensor" type="imu">
             <always_on>true</always_on>

File: description/lidar.xacro (robot description, xacro)
@@ -3,8 +3,8 @@
     <joint name="laser_joint" type="fixed">
         <parent link="chassis"/>
-        <child link="laser_frame"/>
-        <origin xyz="0.4 0 0.13" rpy="0 0 0"/>
+        <child link="laser"/>
+        <origin xyz="0.4 0 0.13" rpy="0 0 3.14"/>
     </joint>
-    <link name="laser_frame">
+    <link name="laser">
         <visual>
             <geometry>
@@ -19,8 +19,8 @@
         </collision>
         <xacro:inertial_cylinder mass="0.1" length="0.04" radius="0.05">
-            <origin xyz="0 0 0" rpy="0 0 0"/>
+            <origin xyz="0 0 0" rpy="0 0 3.14"/>
         </xacro:inertial_cylinder>
     </link>
-    <gazebo reference="laser_frame">
+    <gazebo reference="laser">
         <material>Gazebo/Red</material>
         <sensor name="laser" type="gpu_lidar">

File: description/robot_core.xacro (robot description, xacro)
@@ -6,5 +6,5 @@
     <xacro:property name="chassis_height" value="0.114"/>
     <xacro:property name="chassis_mass" value="1.5"/>
-    <xacro:property name="wheel_radius" value="0.09"/>
+    <xacro:property name="wheel_radius" value="0.045"/>
     <xacro:property name="wheel_thickness" value="0.020"/>
     <xacro:property name="wheel_mass" value="0.07"/>
